File: Kicad/BADGER_v41.kicad_pcb (KiCad board)
At the start: 2 copper layers, 101.6 x 78.7 mm, 117 parts, among them J4 ZIF-40-0.5, P1 PCB, P2 ISP, P3 FTDI, P4 C3SB, P5 JST_3V7, P6 V_IN, P7 UUSB_B, Q1 DMG2301U-7, Q2 2N7002KW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

Commit message: BADGEr added Silk legend and Dimensions PDF Files
Parts:
- A0, A0_3V3, PB2, U5/7, XA3, XB3: footprint I/O -> O:

Commit message: minor mods, no need to regenerate gerbers
Parts:
- A0, A0_3V3, PB2, U5/7, XA3, XB3: value I/O -> IO; footprint O: -> (none)
- AD0, AD1, AD2, AD3, AREF1, H1, H2, H5, H6, PD11, PD12, PD13, PD2, PD4, PD5, PD6, PD7, PD8, PD9, V1, V2: value I/O -> IO
- U1: value MCP9700AT-E/TT -> MCP9700AT
