File: Kicad/BADGER_v41.sch (KiCad schematic (older format))
At the start: 116 parts, among them J4 ZIF-40-0.5, P1 PCB, P2 ISP, P3 FTDI, P4 C3SB, P5 JST_3V7, P6 V_IN, P7 UUSB_B, Q1 DMG2301U-7, Q2 2N7002KW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

Commit message: minor mods, no need to regenerate gerbers
Parts:
- A0, A0_3V3, PB2, U5/7, XA3, XB3: value I/O -> IO; footprint I/O -> IO; symbol I/O -> IO
- AD0, AD1, AD2, AD3, AREF1, PD11, PD12, PD13, PD2, PD4, PD5, PD6, PD7, PD8, PD9, V1, V2: value I/O -> IO; symbol I/O -> IO
- BT1: symbol BATT_HOLDER -> Batt_Holder
- BT2: value BATT_COIN -> Batt_Coin; symbol BATT_COIN -> Batt_Coin
- SD1: value SD_CARD_MICRO -> SD_CARD_Micro; symbol SD_CARD_MICRO -> SD_CARD_Micro
- U1: value MCP9700AT-E/TT -> MCP9700AT; symbol MCP9700AT-E/TT -> MCP9700AT
Changed lines of the file:
@@
 LIBS:power
 LIBS:BADGER_v41-cache
-EELAYER 24 0
+EELAYER 25 0
 EELAYER END
 $Descr A4 11693 8268
@@
 Text Notes 7050 3575 0    30   ~ 0
 PWM : 100 - 300KHz\n50% duty cycle, square wave
-Text Notes 7050 3050 0    30   ~ 0
+Text Notes 7050 3100 0    30   ~ 0
 DISCHARGE: set high for EPD\ndischarge when EPD power off
 Text Notes 625  2225 0    40   ~ 8
@@
 NoConn ~ 2300 3075
 $Comp
-L SD_CARD_MICRO SD1
+L SD_CARD_Micro SD1
 U 1 1 5152F006
 P 1800 2875
 F 0 "SD1" H 1950 3325 40  0000 C CNN
-F 1 "SD_CARD_MICRO" H 2375 3325 40  0000 C CNN
+F 1 "SD_CARD_Micro" H 2375 3325 40  0000 C CNN
 F 2 "SD_Micro_seeed" H 1800 2875 60  0001 C CNN
 F 3 "" H 1800 2875 60  0001 C CNN
@@
 $EndComp
 $Comp
-L MCP9700AT-E/TT U1
+L MCP9700AT U1
 U 1 1 5155C609
 P 1275 1675
 F 0 "U1" H 1275 1725 30  0000 L CNN
-F 1 "MCP9700AT-E/TT" H 1275 1775 30  0000 L CNN
+F 1 "MCP9700AT" H 1275 1775 30  0000 L CNN
 F 2 "SOT23-3-Temp" H 1275 1675 60  0001 C CNN
 F 3 "~" H 1275 1675 60  0000 C CNN
@@
 $EndComp
 $Comp
-L I/O A0_3V3
+L IO A0_3V3
 U 1 1 5159E685
 P 2175 4075
 F 0 "A0_3V3" H 2225 4075 40  0000 L CNN
-F 1 "I/O" H 2175 4020 30  0001 C CNN
-F 2 "I/O" H 2175 4075 60  0001 C CNN
+F 1 "IO" H 2175 4020 30  0001 C CNN
+F 2 "IO" H 2175 4075 60  0001 C CNN
 F 3 "~" H 2175 4075 60  0000 C CNN
 	1    2175 4075
@@
 VCC5V
 $Comp
-L I/O PB2
+L IO PB2
 U 1 1 515FE54A
 P 6650 6750
 F 0 "PB2" H 6625 6800 40  0000 L BNN
-F 1 "I/O" H 6650 6805 30  0001 C CNN
-F 2 "I/O" H 6650 6750 60  0001 C CNN
+F 1 "IO" H 6650 6805 30  0001 C CNN
+F 2 "IO" H 6650 6750 60  0001 C CNN
 F 3 "~" H 6650 6750 60  0000 C CNN
 	1    6650 6750
@@
 SPI_SS
 $Comp
-L BATT_HOLDER BT1
+L Batt_Holder BT1
 U 1 1 51612040
 P 10525 6475
@@
 $EndComp
 $Comp
-L BATT_COIN BT2
+L Batt_Coin BT2
 U 1 1 516122F7
 P 10525 6825
 F 0 "BT2" V 10475 6925 30  0000 L CNN
-F 1 "BATT_COIN" V 10525 6925 30  0000 L CNN
+F 1 "Batt_Coin" V 10525 6925 30  0000 L CNN
 F 2 "CR2032" H 10525 6825 60  0001 C CNN
 F 3 "~" H 10525 6825 60  0000 C CNN
@@
 SPI_SS
 $Comp
-L I/O A0
+L IO A0
 U 1 1 51627367
 P 775 4075
 F 0 "A0" H 825 4075 40  0000 L CNN
-F 1 "I/O" H 775 4020 30  0001 C CNN
-F 2 "I/O" H 775 4075 60  0001 C CNN
+F 1 "IO" H 775 4020 30  0001 C CNN
+F 2 "IO" H 775 4075 60  0001 C CNN
 F 3 "~" H 775 4075 60  0000 C CNN
 	1    775  4075
@@
 $EndComp
 $Comp
-L I/O XB3
+L IO XB3
 U 1 1 5162736D
 P 775 4175
 F 0 "XB3" H 825 4175 40  0000 L CNN
-F 1 "I/O" H 775 4120 30  0001 C CNN
-F 2 "I/O" H 775 4175 60  0001 C CNN
+F 1 "IO" H 775 4120 30  0001 C CNN
+F 2 "IO" H 775 4175 60  0001 C CNN
 F 3 "~" H 775 4175 60  0000 C CNN
 	1    775  4175
@@
 Connection ~ 6775 5350
 $Comp
-L I/O XA3
+L IO XA3
 U 1 1 51645932
 P 2175 4175
 F 0 "XA3" H 2225 4175 40  0000 L CNN
-F 1 "I/O" H 2175 4120 30  0001 C CNN
-F 2 "I/O" H 2175 4175 60  0001 C CNN
+F 1 "IO" H 2175 4120 30  0001 C CNN
+F 2 "IO" H 2175 4175 60  0001 C CNN
 F 3 "~" H 2175 4175 60  0000 C CNN
 	1    2175 4175
@@
 Wire Wire Line
 	7800 2775 7800 2825
-Text Notes 10625 6900 0    30   ~ 0
+Text Notes 10225 6875 0    30   ~ 0
 CR2450\nor\nCR2032
-Text Notes 7100 6525 0    30   ~ 0
+Text Notes 7100 6075 0    30   ~ 0
 7.2V LiPo\n9V Battery\n12V Wall Wart
-Text Notes 7925 6275 0    30   ~ 0
+Text Notes 7925 6325 0    30   ~ 0
 Lanyard\nHoles
 $Comp
-L I/O U5/7
+L IO U5/7
 U 1 1 516E4DF2
 P 2725 5600
 F 0 "U5/7" H 2805 5600 40  0000 L CNN
-F 1 "I/O" H 2725 5545 30  0001 C CNN
-F 2 "I/O" H 2725 5600 60  0001 C CNN
+F 1 "IO" H 2725 5545 30  0001 C CNN
+F 2 "IO" H 2725 5600 60  0001 C CNN
 F 3 "~" H 2725 5600 60  0000 C CNN
 	1    2725 5600
@@
 Text Label 6150 5850 0    40   ~ 0
 UP
-Text Notes 9350 4150 0    30   ~ 0
+Text Notes 9350 4375 0    30   ~ 0
 NOTE : S_LINK (SL1) is bridged [ D2 is bypassed ] when powering the Badge\nfrom the Coin Battery.\nWhen using ANY OTHER power source (Lipo on JST, 5V on USB, 12V Barrel\nsocket etc), Unbridge D2 (remove solder from link SL1).\nThe Coin Battery can then be used as power source for RTC.\nIf RTC is not used,  REMOVE the Coin Battery.
 Text Notes 10825 6200 0    30   ~ 0
@@
 VCC5V
 $Comp
-L I/O AREF1
+L IO AREF1
 U 1 1 51B9C518
 P 6800 1150
 F 0 "AREF1" H 6850 1150 40  0000 L CNN
-F 1 "I/O" H 6800 1095 30  0001 C CNN
+F 1 "IO" H 6800 1095 30  0001 C CNN
 F 2 "Breakout" H 6800 1150 60  0001 C CNN
 F 3 "~" H 6800 1150 60  0000 C CNN
@@
 $EndComp
 $Comp
-L I/O PD13
+L IO PD13
 U 1 1 51B9C51E
 P 6550 1350
 F 0 "PD13" H 6600 1350 40  0000 L CNN
-F 1 "I/O" H 6550 1295 30  0001 C CNN
+F 1 "IO" H 6550 1295 30  0001 C CNN
 F 2 "Breakout" H 6550 1350 60  0001 C CNN
 F 3 "~" H 6550 1350 60  0000 C CNN
@@
 $EndComp
 $Comp
-L I/O PD12
+L IO PD12
 U 1 1 51B9C524
 P 6550 1450
 F 0 "PD12" H 6600 1450 40  0000 L CNN
-F 1 "I/O" H 6550 1395 30  0001 C CNN
+F 1 "IO" H 6550 1395 30  0001 C CNN
 F 2 "Breakout" H 6550 1450 60  0001 C CNN
 F 3 "~" H 6550 1450 60  0000 C CNN
@@
 $EndComp
 $Comp
-L I/O PD11
+L IO PD11
 U 1 1 51B9C52A
 P 6550 1550
 F 0 "PD11" H 6600 1550 40  0000 L CNN
-F 1 "I/O" H 6550 1495 30  0001 C CNN
+F 1 "IO" H 6550 1495 30  0001 C CNN
 F 2 "Breakout" H 6550 1550 60  0001 C CNN
 F 3 "~" H 6550 1550 60  0000 C CNN
@@
 	6125 1850 6400 1850
 $Comp
-L I/O PD9
+L IO PD9
 U 1 1 51B9C78A
 P 6550 1750
 F 0 "PD9" H 6600 1750 40  0000 L CNN
-F 1 "I/O" H 6550 1695 30  0001 C CNN
+F 1 "IO" H 6550 1695 30  0001 C CNN
 F 2 "Breakout" H 6550 1750 60  0001 C CNN
 F 3 "~" H 6550 1750 60  0000 C CNN
@@
 $EndComp
 $Comp
-L I/O PD8
+L IO PD8
 U 1 1 51B9C790
 P 6550 1850
 F 0 "PD8" H 6600 1850 40  0000 L CNN
-F 1 "I/O" H 6550 1795 30  0001 C CNN
+F 1 "IO" H 6550 1795 30  0001 C CNN
 F 2 "Breakout" H 6550 1850 60  0001 C CNN
 F 3 "~" H 6550 1850 60  0000 C CNN
@@
 	6125 2350 6400 2350
 $Comp
-L I/O PD7
+L IO PD7
 U 1 1 51B9C7B9
 P 6550 2050
 F 0 "PD7" H 6600 2050 40  0000 L CNN
-F 1 "I/O" H 6550 1995 30  0001 C CNN
+F 1 "IO" H 6550 1995 30  0001 C CNN
 F 2 "Breakout" H 6550 2050 60  0001 C CNN
 F 3 "~" H 6550 2050 60  0000 C CNN
@@
 $EndComp
 $Comp
-L I/O PD6
+L IO PD6
 U 1 1 51B9C7BF
 P 6550 2150
 F 0 "PD6" H 6600 2150 40  0000 L CNN
-F 1 "I/O" H 6550 2095 30  0001 C CNN
+F 1 "IO" H 6550 2095 30  0001 C CNN
 F 2 "Breakout" H 6550 2150 60  0001 C CNN
 F 3 "~" H 6550 2150 60  0000 C CNN
@@
 $EndComp
 $Comp
-L I/O PD5
+L IO PD5
 U 1 1 51B9C7C5
 P 6550 2250
 F 0 "PD5" H 6600 2250 40  0000 L CNN
-F 1 "I/O" H 6550 2195 30  0001 C CNN
+F 1 "IO" H 6550 2195 30  0001 C CNN
 F 2 "Breakout" H 6550 2250 60  0001 C CNN
 F 3 "~" H 6550 2250 60  0000 C CNN
@@
 $EndComp
 $Comp
-L I/O PD4
+L IO PD4
 U 1 1 51B9C7CC
 P 6550 2350
 F 0 "PD4" H 6600 2350 40  0000 L CNN
-F 1 "I/O" H 6550 2295 30  0001 C CNN
+F 1 "IO" H 6550 2295 30  0001 C CNN
 F 2 "Breakout" H 6550 2350 60  0001 C CNN
 F 3 "~" H 6550 2350 60  0000 C CNN
@@
 	6125 2550 6400 2550
 $Comp
-L I/O PD2
+L IO PD2
 U 1 1 51B9C7E4
 P 6550 2550
 F 0 "PD2" H 6600 2550 40  0000 L CNN
-F 1 "I/O" H 6550 2495 30  0001 C CNN
+F 1 "IO" H 6550 2495 30  0001 C CNN
 F 2 "Breakout" H 6550 2550 60  0001 C CNN
 F 3 "~" H 6550 2550 60  0000 C CNN
@@
 	4025 2250 3750 2250
 $Comp
-L I/O AD3
+L IO AD3
 U 1 1 51B9D67E
 P 3600 2550
 F 0 "AD3" H 3650 2550 40  0000 L CNN
-F 1 "I/O" H 3600 2495 30  0001 C CNN
+F 1 "IO" H 3600 2495 30  0001 C CNN
 F 2 "Breakout" H 3600 2550 60  0001 C CNN
 F 3 "~" H 3600 2550 60  0000 C CNN
@@
 $EndComp
 $Comp
-L I/O AD2
+L IO AD2
 U 1 1 51B9D684
 P 3600 2450
 F 0 "AD2" H 3650 2450 40  0000 L CNN
-F 1 "I/O" H 3600 2395 30  0001 C CNN
+F 1 "IO" H 3600 2395 30  0001 C CNN
 F 2 "Breakout" H 3600 2450 60  0001 C CNN
 F 3 "~" H 3600 2450 60  0000 C CNN
@@
 $EndComp
 $Comp
-L I/O AD1
+L IO AD1
 U 1 1 51B9D68A
 P 3600 2350
 F 0 "AD1" H 3650 2350 40  0000 L CNN
-F 1 "I/O" H 3600 2295 30  0001 C CNN
+F 1 "IO" H 3600 2295 30  0001 C CNN
 F 2 "Breakout" H 3600 2350 60  0001 C CNN
 F 3 "~" H 3600 2350 60  0000 C CNN
@@
 $EndComp
 $Comp
-L I/O AD0
+L IO AD0
 U 1 1 51B9D690
 P 3600 2250
 F 0 "AD0" H 3650 2250 40  0000 L CNN
-F 1 "I/O" H 3600 2195 30  0001 C CNN
+F 1 "IO" H 3600 2195 30  0001 C CNN
 F 2 "Breakout" H 3600 2250 60  0001 C CNN
 F 3 "~" H 3600 2250 60  0000 C CNN
@@
 	3525 2050 4025 2050
 $Comp
-L I/O V1
+L IO V1
 U 1 1 51B9D6B0
 P 3375 2050
 F 0 "V1" H 3425 2050 40  0000 L CNN
-F 1 "I/O" H 3375 1995 30  0001 C CNN
+F 1 "IO" H 3375 1995 30  0001 C CNN
 F 2 "Breakout" H 3375 2050 60  0001 C CNN
 F 3 "~" H 3375 2050 60  0000 C CNN
@@
 	3525 1650 4025 1650
 $Comp
-L I/O V2
+L IO V2
 U 1 1 51B9D6C1
 P 3375 1650
 F 0 "V2" H 3425 1650 40  0000 L CNN
-F 1 "I/O" H 3375 1595 30  0001 C CNN
+F 1 "IO" H 3375 1595 30  0001 C CNN
 F 2 "Breakout" H 3375 1650 60  0001 C CNN
 F 3 "~" H 3375 1650 60  0000 C CNN
